File: DIY_Blackpill.sch (KiCad schematic (older format))
At the start: 34 parts, among them J1 Conn_01x20, J2 Conn_01x20, J3 USB_B_Micro, J4 Conn_02x03_Top_Bottom, J5 Conn_01x04_Male, SW1 SW_SPST, U1 STM32F103C8Tx, U2 FT230XS, U3 TLV70033_SOT353, Y1 8M

Commit message: Switched Footprint of TVL70033
Parts:
- U3: footprint Package_TO_SOT_SMD:SOT-353_SC-70-5_Handsoldering -> SamacSys_Parts:SOT95P280X110-5N
Changed lines of the file:
@@
 F 0 "U3" H 10300 5092 50  0000 C CNN
 F 1 "TLV70033_SOT353" H 10300 5001 50  0000 C CNN
-F 2 "Package_TO_SOT_SMD:SOT-353_SC-70-5_Handsoldering" H 10300 5050 50  0001 C CIN
+F 2 "SamacSys_Parts:SOT95P280X110-5N" H 10300 5050 50  0001 C CIN
 F 3 "http://www.ti.com/lit/ds/symlink/tlv700.pdf" H 10300 4800 50  0001 C CNN
 	1    10300 4750
