File: DIY_Blackpill.kicad_pcb (KiCad board)
At the start: 2 copper layers, 27.9 x 62.2 mm, 34 parts, among them J1 Conn_01x20, J2 Conn_01x20, J3 USB_B_Micro, J4 Conn_02x03_Top_Bottom, J5 Conn_01x04_Male, SW1 SW_SPST, U1 STM32F103C8Tx, U2 FT230XS, U3 TLV70033_SOT353, Y1 8M

Commit message: Switched Footprint of TVL70033
Parts:
- U3: footprint Package_TO_SOT_SMD:SOT-353_SC-70-5_Handsoldering -> SamacSys_Parts:SOT95P280X110-5N
Routing:
- net +3V3: track 187.6 -> 186.3 mm
- net GND: vias 34 -> 35

Commit message: Added way more via's
Routing:
- net GND: vias 35 -> 95
Changed lines of the file:
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@@
     (thickness 1.6)
     (drawings 7)
-    (tracks 498)
+    (tracks 558)
     (zones 0)
     (modules 34)
@@
   (via (at 55.118 40.132) (size 0.8) (drill 0.4) (layers F.Cu B.Cu) (net 2))
   (via (at 61.214 51.816) (size 0.8) (drill 0.4) (layers F.Cu B.Cu) (net 2))
+  (via (at 55.626 47.752) (size 0.8) (drill 0.4) (layers F.Cu B.Cu) (net 2))
+  (via (at 65.786 37.084) (size 0.8) (drill 0.4) (layers F.Cu B.Cu) (net 2))
+  (via (at 64.516 37.084) (size 0.8) (drill 0.4) (layers F.Cu B.Cu) (net 2))
+  (via (at 77.216 37.084) (size 0.8) (drill 0.4) (layers F.Cu B.Cu) (net 2))
+  (via (at 52.324 36.83) (size 0.8) (drill 0.4) (layers F.Cu B.Cu) (net 2))
+  (via (at 53.848 36.83) (size 0.8) (drill 0.4) (layers F.Cu B.Cu) (net 2))
+  (via (at 55.626 36.83) (size 0.8) (drill 0.4) (layers F.Cu B.Cu) (net 2))
+  (via (at 57.404 36.83) (size 0.8) (drill 0.4) (layers F.Cu B.Cu) (net 2))
+  (via (at 51.816 45.212) (size 0.8) (drill 0.4) (layers F.Cu B.Cu) (net 2))
+  (via (at 51.816 42.926) (size 0.8) (drill 0.4) (layers F.Cu B.Cu) (net 2))
+  (via (at 52.07 40.132) (size 0.8) (drill 0.4) (layers F.Cu B.Cu) (net 2))
+  (via (at 74.93 37.084) (size 0.8) (drill 0.4) (layers F.Cu B.Cu) (net 2))
+  (via (at 72.898 37.084) (size 0.8) (drill 0.4) (layers F.Cu B.Cu) (net 2))
+  (via (at 74.93 38.862) (size 0.8) (drill 0.4) (layers F.Cu B.Cu) (net 2))
+  (via (at 77.216 42.672) (size 0.8) (drill 0.4) (layers F.Cu B.Cu) (net 2))
+  (via (at 61.214 78.994) (size 0.8) (drill 0.4) (layers F.Cu B.Cu) (net 2))
+  (via (at 58.928 78.994) (size 0.8) (drill 0.4) (layers F.Cu B.Cu) (net 2))
+  (via (at 57.15 79.756) (size 0.8) (drill 0.4) (layers F.Cu B.Cu) (net 2))
+  (via (at 56.642 81.788) (size 0.8) (drill 0.4) (layers F.Cu B.Cu) (net 2))
+  (via (at 56.134 84.836) (size 0.8) (drill 0.4) (layers F.Cu B.Cu) (net 2))
+  (via (at 54.61 87.122) (size 0.8) (drill 0.4) (layers F.Cu B.Cu) (net 2))
+  (via (at 56.134 87.122) (size 0.8) (drill 0.4) (layers F.Cu B.Cu) (net 2))
+  (via (at 57.404 87.122) (size 0.8) (drill 0.4) (layers F.Cu B.Cu) (net 2))
+  (via (at 57.404 84.836) (size 0.8) (drill 0.4) (layers F.Cu B.Cu) (net 2))
+  (via (at 58.674 82.55) (size 0.8) (drill 0.4) (layers F.Cu B.Cu) (net 2))
+  (via (at 60.96 83.82) (size 0.8) (drill 0.4) (layers F.Cu B.Cu) (net 2))
+  (via (at 59.182 85.852) (size 0.8) (drill 0.4) (layers F.Cu B.Cu) (net 2))
+  (via (at 62.738 85.344) (size 0.8) (drill 0.4) (layers F.Cu B.Cu) (net 2))
+  (via (at 65.024 87.63) (size 0.8) (drill 0.4) (layers F.Cu B.Cu) (net 2))
+  (via (at 66.548 86.106) (size 0.8) (drill 0.4) (layers F.Cu B.Cu) (net 2))
+  (via (at 64.008 83.566) (size 0.8) (drill 0.4) (layers F.Cu B.Cu) (net 2))
+  (via (at 57.912 94.996) (size 0.8) (drill 0.4) (layers F.Cu B.Cu) (net 2))
+  (via (at 59.436 93.726) (size 0.8) (drill 0.4) (layers F.Cu B.Cu) (net 2))
+  (via (at 57.658 89.916) (size 0.8) (drill 0.4) (layers F.Cu B.Cu) (net 2))
+  (via (at 55.626 91.948) (size 0.8) (drill 0.4) (layers F.Cu B.Cu) (net 2))
+  (via (at 66.04 72.39) (size 0.8) (drill 0.4) (layers F.Cu B.Cu) (net 2))
+  (via (at 67.056 71.628) (size 0.8) (drill 0.4) (layers F.Cu B.Cu) (net 2))
+  (via (at 77.978 59.182) (size 0.8) (drill 0.4) (layers F.Cu B.Cu) (net 2))
+  (via (at 77.978 56.642) (size 0.8) (drill 0.4) (layers F.Cu B.Cu) (net 2))
+  (via (at 77.724 51.816) (size 0.8) (drill 0.4) (layers F.Cu B.Cu) (net 2))
+  (via (at 68.834 46.736) (size 0.8) (drill 0.4) (layers F.Cu B.Cu) (net 2))
+  (via (at 68.834 44.704) (size 0.8) (drill 0.4) (layers F.Cu B.Cu) (net 2))
+  (via (at 68.834 50.292) (size 0.8) (drill 0.4) (layers F.Cu B.Cu) (net 2))
+  (via (at 68.834 51.816) (size 0.8) (drill 0.4) (layers F.Cu B.Cu) (net 2))
+  (via (at 64.516 56.388) (size 0.8) (drill 0.4) (layers F.Cu B.Cu) (net 2))
+  (via (at 63.754 58.166) (size 0.8) (drill 0.4) (layers F.Cu B.Cu) (net 2))
+  (via (at 59.69 56.134) (size 0.8) (drill 0.4) (layers F.Cu B.Cu) (net 2))
+  (via (at 59.69 52.832) (size 0.8) (drill 0.4) (layers F.Cu B.Cu) (net 2))
+  (via (at 51.816 54.356) (size 0.8) (drill 0.4) (layers F.Cu B.Cu) (net 2))
+  (via (at 51.816 49.022) (size 0.8) (drill 0.4) (layers F.Cu B.Cu) (net 2))
+  (via (at 51.816 64.516) (size 0.8) (drill 0.4) (layers F.Cu B.Cu) (net 2))
+  (via (at 51.816 69.596) (size 0.8) (drill 0.4) (layers F.Cu B.Cu) (net 2))
+  (via (at 51.562 74.676) (size 0.8) (drill 0.4) (layers F.Cu B.Cu) (net 2))
+  (via (at 51.816 79.756) (size 0.8) (drill 0.4) (layers F.Cu B.Cu) (net 2))
+  (via (at 51.816 82.042) (size 0.8) (drill 0.4) (layers F.Cu B.Cu) (net 2))
+  (via (at 65.532 42.926) (size 0.8) (drill 0.4) (layers F.Cu B.Cu) (net 2))
+  (via (at 64.77 67.31) (size 0.8) (drill 0.4) (layers F.Cu B.Cu) (net 2))
+  (via (at 64.516 69.342) (size 0.8) (drill 0.4) (layers F.Cu B.Cu) (net 2))
+  (via (at 64.77 90.17) (size 0.8) (drill 0.4) (layers F.Cu B.Cu) (net 2))
+  (via (at 64.77 92.71) (size 0.8) (drill 0.4) (layers F.Cu B.Cu) (net 2))
   (segment (start 71.374 43.924) (end 70.8988 44.3992) (width 0.25) (layer F.Cu) (net 3))
   (segment (start 66.182 40.675998) (end 67.487998 39.37) (width 0.25) (layer F.Cu) (net 3))
